File: opto-interface-arduino/hardware/opto-interface.kicad_pcb (KiCad board)
At the start: 2 copper layers, 0 parts

Commit message: Move current Kicad files to hardware subdirectory.  Update tripod QR plate to be slightly less wide.
Parts:
- added C1, C2: 0u1F, Capacitors_ThroughHole:C_Disc_D6_P5, F.Cu at (148.5, 105.0)
- added C3, C4: 2u2F, Discret:CP5, F.Cu at (148.5, 105.0)
- added P1: CONN_02X06, Pin_Headers:Pin_Header_Straight_2x06, F.Cu at (148.5, 105.0)
- added R1, R2: 100kR, Resistors_SMD:R_0805_HandSoldering, F.Cu at (148.5, 105.0)
- added R3: 390R, Resistors_SMD:R_0805_HandSoldering, F.Cu at (148.5, 105.0)
- added SHIELD1: ARDUINO_SHIELD, arduino_shields:ARDUINO SHIELD, F.Cu at (148.5, 105.0)
- added U1: LM7805, TO_SOT_Packages_THT:TO-220_Neutral123_Horizontal_LargePads, F.Cu at (148.5, 105.0)
- added U2: LM7905, TO_SOT_Packages_THT:TO-220_Neutral123_Horizontal_LargePads, F.Cu at (148.5, 105.0)
Other:
- net class Default: clearance 0.1524 -> 0.2; trace_width 0.1524 -> 0.25; via_dia 0.6096 -> 0.6; via_drill 0.3302 -> 0.4
- rule pad_to_mask_clearance: 0.05 -> 0
- rule trace_clearance: 0.1524 -> 0.2
- rule trace_min: 0.1524 -> 0.2
- rule via_min_drill: 0.3302 -> 0.3
- rule via_min_size: 0.6096 -> 0.4
